File: Prop.kicad_pcb (KiCad board)
At the start: 2 copper layers, 63.5 x 63.5 mm, 87 parts, among them J1 1984989, J10 1984989, J11 1984989, J12 1984989, J13 1984989, J14 1984989, J15 Anderson_Powerpole, J16 1984989, J2 1984989, J3 1984989, J4 1984989, J5 CAS_stacking, J6 1984989, J7 1984989, J8 1984989, J9 1984989, U10 LM386, U11 LM386, U12 LM386, U13 LM386, U1301 MAX6675ISA+, U14 LM386, U15 MCP3008, U16 LM386, U2 MAX6675ISA+, U3 MAX6675ISA+, U4 LM386, U5 MCP3008, U6 L298P, U7 SN74LVC8T245DBR, U8 SN74LVC2GU04DCKR, U9 LM386

Commit message: split board into 3
Parts:
- added J5: CAS_stacking, star-common-lib:CAS_physical, F.Cu at (27.9, 55.9)
- added J5: CAS_stacking, star-common-lib:CAS_physical, F.Cu at (204.5, 54.6)
- moved R5 206.3 mm to (39.9, 74.9)
- moved R8 202.1 mm to (39.9, 78.7)
- moved C12 200.4 mm to (44.0, 74.9), turned to 180 degrees
- moved R4 199.3 mm to (38.1, 93.5), turned to 270 degrees
- moved C11 197.0 mm to (40.6, 96.5), turned to 180 degrees
- moved C8 196.1 mm to (53.3, 72.4), turned to 180 degrees
- moved C19 192.0 mm to (53.3, 76.7), turned to 90 degrees
- moved C18 189.3 mm to (57.6, 73.7), turned to 180 degrees
- moved C9 184.6 mm to (43.7, 100.3), turned to 180 degrees
- moved R10 183.5 mm to (53.3, 99.8), turned to 90 degrees
- moved R13 182.8 mm to (38.1, 89.7), turned to 270 degrees
- moved U2 181.6 mm to (80.0, 81.3)
- moved R9 181.5 mm to (40.6, 89.7), turned to 270 degrees
- moved R12 180.4 mm to (39.9, 82.5)
- moved R7 180.4 mm to (48.3, 74.9)
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