File: prop/prop.kicad_pcb (KiCad board)
At the start: 4 copper layers, 63.5 x 63.5 mm, 89 parts, among them J1 1984989, J10 1984989, J1001 CAS_stacking, J11 1984989, J12 1984989, J13 1984989, J14 1984989, J16 1984989, J2 1984989, J3 1984989, J4 1984989, J5 Conn_01x02, J6 1984989, J7 1984989, J8 1984989, J9 1984989, U10 LM386, U11 LM386, U12 LM386, U13 LM386, U1301 MAX6675ISA+, U14 LM386, U15 MCP3008, U16 LM386, U2 MAX6675ISA+, U3 MAX6675ISA+, U4 LM386, U5 MCP3008, U6 L298P, U7 SN74LVC8T245DBR, U8 SN74LVC2GU04DCKR, U9 LM386

Commit message: working on left board
Routing:
- net GND: track 56.2 -> 167.4 mm, vias 0 -> 40
- net +5V: track 37.6 -> 81.9 mm, vias 0 -> 19
- net /SPIO_MOSI: track 0.00 -> 28.5 mm
- net Net-(R10-Pad2): track 0.00 -> 15.4 mm
- net Net-(C13-Pad1): track 0.00 -> 14.9 mm
- net /SPI0_MISO: track 0.00 -> 12.1 mm
- net Net-(R4-Pad1): track 0.00 -> 11.7 mm
- net Net-(C19-Pad2): track 0.00 -> 11.6 mm
- net Net-(R3-Pad1): track 0.00 -> 10.7 mm
- net /SPIO_SCK: track 0.00 -> 10.7 mm
- net Net-(C6-Pad2): track 0.00 -> 9.16 mm
- net Net-(C14-Pad2): track 0.00 -> 9.09 mm
- net Net-(R16-Pad2): track 0.00 -> 7.02 mm
- net Net-(C8-Pad2): track 0.00 -> 6.36 mm
- net Net-(C19-Pad1): track 0.00 -> 5.07 mm
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Other:
- rule via_min_drill: 0.3 -> 0.254
- rule via_min_size: 0.4 -> 0.5588

Commit message: more layout on middle board
Routing:
- net GND: track 167.4 -> 248.3 mm, vias 40 -> 57
- net /PWM3: track 0.00 -> 67.9 mm, vias 0 -> 2
- net /SPI0_MISO: track 12.1 -> 80.0 mm, vias 0 -> 4
- net +24V: track 0.00 -> 61.6 mm
- net /PWM2_33: track 0.00 -> 54.0 mm, vias 0 -> 2
- net /Servo_Control/Sol1: track 0.00 -> 49.5 mm, vias 0 -> 4
- net /PWM2: track 0.00 -> 47.8 mm
- net /Sol1_33: track 0.00 -> 46.4 mm, vias 0 -> 2
- net Net-(R1-Pad2): track 0.00 -> 44.9 mm
- net /PWM1: track 0.00 -> 44.4 mm, vias 0 -> 2
- net /Servo_Control/Sol2Lead2: track 0.00 -> 42.5 mm, vias 0 -> 2
- net /CS1: track 0.00 -> 39.8 mm, vias 0 -> 2
- net /ADC_Amp/aData0: track 0.00 -> 37.7 mm
- net /Servo_Control/Sol1': track 0.00 -> 37.6 mm
- net /Servo_Control/Sol2: track 0.00 -> 37.4 mm, vias 0 -> 2
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
Commit message: mostly done with routing on all 3 boards
Parts:
- removed the J1001 at (31.1, 54.7)
- removed the J1001 at (204.5, 54.6)
- added J1001: CAS_stacking, star-common-lib:CAS_physical, F.Cu at (34.7, 54.5)
- added J1001: CAS_stacking, star-common-lib:CAS_physical, F.Cu at (201.7, 54.9)
- moved J8 3.57 mm to (82.7, 111.3)
- moved C10 3.57 mm to (60.3, 80.6)
- moved C12 3.57 mm to (55.9, 101.2)
- moved C8 3.57 mm to (52.6, 95.6)
- moved J1 3.57 mm to (50.3, 61.1)
- moved J2 3.57 mm to (66.4, 61.1)
- moved J7 3.57 mm to (66.5, 111.3)
- moved R12 3.57 mm to (43.7, 94.9)
- moved R15 3.57 mm to (64.6, 94.9)
- moved R8 3.57 mm to (64.7, 77.2)
- moved R5 3.57 mm to (55.9, 95.6)
- moved C1301 3.57 mm to (43.4, 70.1)
- moved C14 3.57 mm to (64.9, 80.6)
- moved C15 3.57 mm to (81.1, 80.5)
- moved C16 3.57 mm to (52.7, 101.1)
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Routing:
- net /PWM1_33: track 0.00 -> 83.6 mm, vias 0 -> 4
- net /Sol2_33: track 0.00 -> 56.0 mm, vias 0 -> 2
- net /PWM3_33: track 0.00 -> 50.4 mm, vias 0 -> 4
- net /CS4: track 0.00 -> 49.8 mm, vias 0 -> 2
- net /SPIO_SCK: track 32.7 -> 82.0 mm, vias 0 -> 2
- net +3V3: track 0.65 -> 40.7 mm, vias 0 -> 2
- net /CS5: track 0.00 -> 30.8 mm
- net +5V: track 119.1 -> 121.7 mm, vias 29 -> 30
