File: prop/prop.kicad_pcb (KiCad board)
At the start: 2 copper layers, 63.5 x 63.5 mm, 89 parts, among them J1 1984989, J10 1984989, J1001 CAS_stacking, J11 1984989, J12 1984989, J13 1984989, J14 1984989, J16 1984989, J2 1984989, J3 1984989, J4 1984989, J5 Conn_01x02, J6 1984989, J7 1984989, J8 1984989, J9 1984989, U10 LM386, U11 LM386, U12 LM386, U13 LM386, U1301 MAX6675ISA+, U14 LM386, U15 MCP3008, U16 LM386, U2 MAX6675ISA+, U3 MAX6675ISA+, U4 LM386, U5 MCP3008, U6 L298P, U7 SN74LVC8T245DBR, U8 SN74LVC2GU04DCKR, U9 LM386

Commit message: started routing
Parts:
- moved J9 0.89 mm to (148.8, 111.4)
- moved C18 0.72 mm to (85.9, 101.9)
- moved R17 0.72 mm to (85.9, 96.4)
- moved C11 0.51 mm to (72.9, 78.1)
- moved C17 0.51 mm to (65.3, 96.4)
- moved R5 0.51 mm to (52.3, 96.4)
- moved R9 0.51 mm to (65.8, 75.6)
- moved J1 0.51 mm to (46.7, 61.5)
- moved C10 0.51 mm to (56.7, 81.4)
- moved C12 0.51 mm to (52.3, 102.0)
- moved C13 0.51 mm to (68.5, 101.9)
- moved C1301 0.51 mm to (39.9, 70.9)
- moved C14 0.51 mm to (61.3, 81.4)
- moved C15 0.51 mm to (77.6, 81.3)
- moved C16 0.51 mm to (49.1, 101.9)
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Routing:
- net +5V: track 0.00 -> 337.3 mm
- net /Servo_Control/Sol1: track 0.00 -> 69.7 mm, vias 0 -> 3
- net +24V: track 0.00 -> 55.5 mm
- net /SPI0_MISO: track 0.00 -> 46.3 mm, vias 0 -> 2
- net Net-(C24-Pad2): track 0.00 -> 44.8 mm
- net /ADC_Amp_Extra/Data0: track 0.00 -> 42.6 mm
- net Net-(C26-Pad2): track 0.00 -> 29.5 mm
- net /ADC_Amp_Extra/aData0: track 0.00 -> 27.6 mm, vias 0 -> 2
- net /ADC_Amp_Extra/aData1: track 0.00 -> 26.7 mm, vias 0 -> 2
- net /ADC_Amp_Extra/Data1: track 0.00 -> 26.7 mm, vias 0 -> 2
- net Net-(R22-Pad1): track 0.00 -> 25.4 mm
- net /ADC_Amp_Extra/aData2: track 0.00 -> 24.6 mm, vias 0 -> 2
- net /ADC_Amp_Extra/Data2: track 0.00 -> 21.0 mm, vias 0 -> 2
- net Net-(C25-Pad2): track 0.00 -> 19.8 mm, vias 0 -> 2
- net Net-(C23-Pad1): track 0.00 -> 19.2 mm
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
Commit message: started routing
Routing:
- net +5V: track 337.3 -> 577.5 mm
- net /ADC_Amp/aData1: track 0.00 -> 30.6 mm, vias 0 -> 2
- net Net-(R8-Pad2): track 0.00 -> 28.4 mm, vias 0 -> 2
- net Net-(R10-Pad2): track 0.00 -> 27.2 mm
- net Net-(C7-Pad2): track 0.00 -> 20.5 mm, vias 0 -> 2
- net Net-(R4-Pad1): track 0.00 -> 19.5 mm, vias 0 -> 2
- net Net-(C11-Pad1): track 0.00 -> 19.4 mm, vias 0 -> 2
- net Net-(C15-Pad2): track 0.00 -> 18.3 mm, vias 0 -> 2
- net Net-(C11-Pad2): track 0.00 -> 13.3 mm
- net /ADC_Amp/Data1: track 0.00 -> 12.1 mm

Commit message: Connected power wires.
Other:
- net class Default removed
