File: prop/Prop_PCB_2.kicad_pcb (KiCad board)
At the start: 2 copper layers, 63.5 x 63.5 mm, 47 parts, among them J1 1984989, J2 1984989, J3 1984989, J4 1984989, J5 1984989, J6 1984989, J7 CAS_stacking, U1 LM386, U2 LM386, U3 LM386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

Commit message: finished routing
Parts:
- moved J3 174.6 mm to (196.5, 43.2), turned to 180 degrees
- moved J5 169.4 mm to (196.6, 94.0), turned to 0 degrees
- moved R7 167.3 mm to (203.2, 81.9), turned to 90 degrees
- moved R8 166.7 mm to (203.2, 76.2), turned to 90 degrees
- moved R12 162.7 mm to (199.6, 84.5), turned to 180 degrees
- moved C2 161.2 mm to (203.8, 54.6), turned to -90 degrees
- moved C6 160.6 mm to (199.5, 52.1), turned to 180 degrees
- moved U4 158.8 mm to (197.5, 79.4), turned to 180 degrees
- moved R10 157.9 mm to (194.9, 52.1), turned to 0 degrees
- moved C8 156.8 mm to (195.1, 84.5), turned to 0 degrees
- moved C10 155.1 mm to (203.8, 61.6), turned to 90 degrees
- moved U2 154.0 mm to (197.5, 57.1), turned to 0 degrees
- moved R3 153.9 mm to (191.1, 54.6), turned to -90 degrees
- moved J2 152.4 mm to (180.3, 43.2), turned to 180 degrees
- moved C4 151.9 mm to (191.1, 81.9), turned to 90 degrees
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Routing:
- net GND: track 0.00 -> 263.9 mm, vias 0 -> 17
- net +5V: track 0.00 -> 48.1 mm, vias 0 -> 13
- net SPI0_MISO: track 0.00 -> 40.1 mm, vias 0 -> 4
- net SPI0_SCK: track 0.00 -> 33.7 mm, vias 0 -> 4
- net CS1: track 0.00 -> 31.0 mm, vias 0 -> 2
- net SPI0_MOSI: track 0.00 -> 29.4 mm, vias 0 -> 2
- net Data1: track 0.00 -> 24.9 mm
- net CS3: track 0.00 -> 22.7 mm, vias 0 -> 2
- net Data0: track 0.00 -> 20.3 mm, vias 0 -> 2
- net Data4: track 0.00 -> 18.7 mm, vias 0 -> 2
- net CS2: track 0.00 -> 17.5 mm, vias 0 -> 2
- net aData3: track 0.00 -> 14.2 mm
- net aData2: track 0.00 -> 14.1 mm
- net Data3: track 0.00 -> 13.9 mm, vias 0 -> 2
- net aData4: track 0.00 -> 13.7 mm
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- added copper zone on In2.Cu, net +5V
- added copper zone on In1.Cu, net GND
Other:
- copper layers 2 -> 4

Commit message: fixed outstanding routing errors
Routing:
- net GND: track 263.9 -> 270.8 mm, vias 17 -> 18
- net +5V: track 48.1 -> 51.9 mm, vias 13 -> 14
- net SPI0_SCK: track 33.7 -> 36.0 mm, vias 4 -> 3
- net Data4: track 18.7 -> 20.6 mm
- net SPI0_MISO: track 40.1 -> 38.6 mm, vias 4 -> 2
- net Data3: track 13.9 -> 14.4 mm

Commit message: added STAR and BCA logos
Parts:
- added Ref**: Val**, star-common-lib:star_fancy, F.Cu at (193.3, 65.3)
- added Ref**: Val**, star-common-lib:bac, F.Cu at (200.9, 71.6)
Routing:
- net SPI0_SCK: track 36.0 -> 35.2 mm
- net GND: track 270.8 -> 270.1 mm
- added copper zone on F.Cu, net GND

Commit message: added silkscreen labels
Other:
- board text added: "+5V"
- board text added: "GND"
- board text added: "LC1_Data"
- board text added: "PT1_Data"
- board text added: "PT2_Data"
- board text added: "PT3_Data"
- board text added: "PT4_Data"
- board text added: "TC1+"
- board text added: "TC1-"
- board text added: "TC2+"
- board text added: "TC2-"
Changed lines of the file:
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@@
     (property "Sheetname" "")
     (attr smd)
-    (fp_text reference "R15" (at 0 -1.43) (layer "F.SilkS")
+    (fp_text reference "R15" (at -3.746 0) (layer "F.SilkS")
       (effects (font (size 1 1) (thickness 0.15)))
     )
@@
     (property "Sheetname" "")
     (attr smd)
-    (fp_text reference "U6" (at 1.524 -6.604) (layer "F.SilkS")
+    (fp_text reference "U6" (at 3.81 -4.826) (layer "F.SilkS")
       (effects (font (size 1 1) (thickness 0.15)))
     )
@@
     (property "Sheetname" "")
     (attr smd)
-    (fp_text reference "R9" (at 0 -1.43) (layer "F.SilkS")
+    (fp_text reference "R9" (at -2.54 -0.254) (layer "F.SilkS")
       (effects (font (size 1 1) (thickness 0.15)))
     )
@@
     (property "Sheetname" "")
     (attr through_hole)
-    (fp_text reference "J6" (at -4.318 -7.874) (layer "F.SilkS")
+    (fp_text reference "J6" (at -8.128 -8.636) (layer "F.SilkS")
       (effects (font (size 1 1) (thickness 0.015)))
     )
@@
     (property "Sheetname" "")
     (attr through_hole)
-    (fp_text reference "J2" (at -4.825 -7.693) (layer "F.SilkS")
+    (fp_text reference "J2" (at -5.334 -9.398) (layer "F.SilkS")
       (effects (font (size 1 1) (thickness 0.015)))
     )
@@
     (property "Sheetname" "")
     (attr through_hole)
-    (fp_text reference "J3" (at -6.095 -7.82) (layer "F.SilkS")
+    (fp_text reference "J3" (at -6.731 -9.144) (layer "F.SilkS")
       (effects (font (size 1 1) (thickness 0.015)))
     )
@@
       (effects (font (size 0.8 0.8) (thickness 0.15)) (justify left))
     )
-    (fp_text user "BOARD:" (at 9.051 61) (layer "F.SilkS")
-      (effects (font (size 0.8 0.8) (thickness 0.15)) (justify left))
-    )
     (fp_text user "A1|A2" (at 2.54 10.16) (layer "F.SilkS")
       (effects (font (size 0.8 0.8) (thickness 0.15)))
@@
     (property "Sheetname" "")
     (attr smd)
-    (fp_text reference "R10" (at 0 -1.43) (layer "F.SilkS")
+    (fp_text reference "R10" (at -4.699 0.254) (layer "F.SilkS")
       (effects (font (size 1 1) (thickness 0.15)))
     )
@@
     (property "Sheetname" "")
     (attr smd)
-    (fp_text reference "R12" (at 0 -1.43) (layer "F.SilkS")
+    (fp_text reference "R12" (at -2.35 -0.127) (layer "F.SilkS")
       (effects (font (size 1 1) (thickness 0.15)))
     )
@@
     (property "Sheetname" "")
     (attr smd)
-    (fp_text reference "R11" (at 0 -1.43) (layer "F.SilkS")
+    (fp_text reference "R11" (at -2.413 -0.381) (layer "F.SilkS")
       (effects (font (size 1 1) (thickness 0.15)))
     )
@@
     )
   )
+  (gr_text "+5V" (at 170.18 50.038 180) (layer "F.SilkS")
+    (effects (font (size 0.75 0.75) (thickness 0.15)))
+  )
+  (gr_text "+5V" (at 174.244 86.868) (layer "F.SilkS")
+    (effects (font (size 0.75 0.75) (thickness 0.15)))
+  )
+  (gr_text "+5V" (at 185.928 50.038 180) (layer "F.SilkS")
+    (effects (font (size 0.75 0.75) (thickness 0.15)))
+  )
+  (gr_text "GND" (at 174.498 50.038 180) (layer "F.SilkS")
+    (effects (font (size 0.75 0.75) (thickness 0.15)))
+  )
+  (gr_text "PT3_Data" (at 198.374 86.868) (layer "F.SilkS")
+    (effects (font (size 0.75 0.75) (thickness 0.15)))
+  )
+  (gr_text "PT2_Data" (at 182.372 86.868) (layer "F.SilkS")
+    (effects (font (size 0.75 0.75) (thickness 0.15)))
+  )
+  (gr_text "TC1-" (at 163.068 86.868) (layer "F.SilkS")
+    (effects (font (size 0.75 0.75) (thickness 0.15)))
+  )
+  (gr_text "GND" (at 167.386 50.038 180) (layer "F.SilkS")
+    (effects (font (size 0.75 0.75) (thickness 0.15)))
+  )
+  (gr_text "GND" (at 190.754 50.038 180) (layer "F.SilkS")
+    (effects (font (size 0.75 0.75) (thickness 0.15)))
+  )
+  (gr_text "PT4_Data" (at 163.322 50.038 180) (layer "F.SilkS")
+    (effects (font (size 0.75 0.75) (thickness 0.15)))
+  )
+  (gr_text "GND" (at 159.004 50.038 180) (layer "F.SilkS")
+    (effects (font (size 0.75 0.75) (thickness 0.15)))
+  )
+  (gr_text "PT1_Data" (at 194.818 50.038 180) (layer "F.SilkS")
+    (effects (font (size 0.75 0.75) (thickness 0.15)))
+  )
+  (gr_text "+5V" (at 202.184 50.038 180) (layer "F.SilkS")
+    (effects (font (size 0.75 0.75) (thickness 0.15)))
+  )
+  (gr_text "GND" (at 199.136 50.038 180) (layer "F.SilkS")
+    (effects (font (size 0.75 0.75) (thickness 0.15)))
+  )
+  (gr_text "GND" (at 202.438 86.868) (layer "F.SilkS")
+    (effects (font (size 0.75 0.75) (thickness 0.15)))
+  )
+  (gr_text "LC1_Data" (at 178.816 50.038 180) (layer "F.SilkS")
+    (effects (font (size 0.75 0.75) (thickness 0.15)))
+  )
+  (gr_text "TC2-" (at 169.926 86.868) (layer "F.SilkS")
+    (effects (font (size 0.75 0.75) (thickness 0.15)))
+  )
+  (gr_text "GND" (at 177.8 86.868) (layer "F.SilkS")
+    (effects (font (size 0.75 0.75) (thickness 0.15)))
+  )
+  (gr_text "GND" (at 186.436 86.868) (layer "F.SilkS")
+    (effects (font (size 0.75 0.75) (thickness 0.15)))
+  )
+  (gr_text "GND" (at 194.056 86.868) (layer "F.SilkS")
+    (effects (font (size 0.75 0.75) (thickness 0.15)))
+  )
+  (gr_text "TC1+" (at 159.258 86.868) (layer "F.SilkS")
+    (effects (font (size 0.75 0.75) (thickness 0.15)))
+  )
+  (gr_text "+5V" (at 190.5 86.868) (layer "F.SilkS")
+    (effects (font (size 0.75 0.75) (thickness 0.15)))
+  )
+  (gr_text "TC2+" (at 166.624 86.868) (layer "F.SilkS")
+    (effects (font (size 0.75 0.75) (thickness 0.15)))
+  )
+  (gr_text "GND" (at 183.134 50.038 180) (layer "F.SilkS")
+    (effects (font (size 0.75 0.75) (thickness 0.15)))
+  )
   (segment (start 210.625 52.6551) (end 208.625 52.6551) (width 0.508) (layer "F.Cu") (net 1))
