File: prop/Prop_PCB_3.kicad_pcb (KiCad board)
At the start: 4 copper layers, 63.5 x 63.5 mm, 26 parts, among them J1 1984989, J2 1984989, J3 1984989, J4 CAS_stacking, U1 LM386, U2 LM386, U3 MCP3008, U4 LM386

Commit message: finalized board
Parts:
- added G***: LOGO, star-common-lib:star_8x7, F.Cu at (118.0, 100.5)
- added Ref**: Val**, star-common-lib:bac, F.Cu at (117.0, 110.2)
- moved J3 53.8 mm to (115.2, 59.8)
- moved C7 22.8 mm to (115.0, 87.4)
- moved C1 21.5 mm to (99.0, 87.4)
- moved R7 21.1 mm to (110.2, 76.4)
- moved R2 20.4 mm to (94.2, 82.9)
- moved R1 20.0 mm to (94.2, 76.2)
- moved R5 19.3 mm to (99.0, 75.4)
- moved U1 19.3 mm to (101.3, 81.8)
- moved C3 18.8 mm to (104.2, 76.2), turned to 90 degrees
- moved C9 18.6 mm to (119.5, 87.4)
- moved U3 18.2 mm to (101.2, 102.5)
- moved R8 17.7 mm to (110.2, 82.8)
- moved R9 17.4 mm to (115.0, 75.6)
- moved U4 17.4 mm to (117.3, 81.8)
- moved C8 17.0 mm to (120.2, 76.2), turned to 90 degrees
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Routing:
- net +5V: track 125.1 -> 22.3 mm, vias 0 -> 7
- net SPI0_SCK: track 0.00 -> 65.2 mm
- net CS5: track 0.00 -> 62.5 mm
- net SPI0_MISO: track 0.00 -> 51.0 mm
- net SPI0_MOSI: track 0.00 -> 50.0 mm
- net GND: track 55.9 -> 87.0 mm, vias 0 -> 11
- net aData2: track 0.00 -> 17.7 mm
- net Data0: track 25.8 -> 12.3 mm
- net Data1: track 9.47 -> 19.7 mm
- net Net-(C7-Pad2): track 0.00 -> 8.73 mm
- net Data2: track 35.3 -> 29.1 mm
- net Net-(C5-Pad2): track 9.47 -> 3.97 mm
- net Net-(R1-Pad2): track 5.02 -> 10.0 mm
- net Net-(R3-Pad2): track 5.51 -> 10.0 mm
- net Net-(R7-Pad2): track 5.23 -> 9.68 mm
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- added copper zone on In2.Cu, net +5V
- added copper zone on B.Cu, net GND
- added copper zone on F.Cu, net GND
- added copper zone on In1.Cu, net GND
Other:
- board text added: "LC Connector"
- board text added: "PT Connector"
